File: z80-cpu.kicad_pcb (KiCad board)
At the start: 2 copper layers, 99.1 x 49.9 mm, 25 parts, among them J1 RC2014 Bus, J3 Conn_02x09_Odd_Even, Q1 2N3904, SW1 RESET, U1 Z80 CPU, U2 NE555, U3 74HCT393, X1 ACO-7.3728MHz

Commit message: Fixed missing reset pullup, and slightly broken schematic after changing header labels. Rev 2
Parts:
- added R4: 10k, Resistor_THT:R_Axial_DIN0207_L6.3mm_D2.5mm_P10.16mm_Horizontal, F.Cu at (154.3, 71.1)
- C7: value 10u -> 10uF
- J1: value RC2014 Bus -> RC2014_Bus
- Q1: value 2N3904 -> 2N3904-AP
- moved R6 1.27 mm to (160.7, 71.1)
- moved R7 1.27 mm to (163.8, 71.1)
- moved R5 1.27 mm to (157.5, 71.1)
- moved R8 1.27 mm to (167.0, 71.1)
- renumbered R4 to R5, R5 to R6, R6 to R7, R7 to R8
Connections:
- net +5V renamed VCC
- net /a0 renamed A0
- net /a1 renamed A1
- net /a10 renamed A10
- net /a11 renamed A11
- net /a12 renamed A12
- net /a13 renamed A13
- net /a14 renamed A14
- net /a15 renamed A15
- net /a2 renamed A2
- net /a3 renamed A3
- net /a4 renamed A4
- net /a5 renamed A5
- net /a6 renamed A6
- net /a7 renamed A7
- net /a8 renamed A8
- net /a9 renamed A9
- net /clk renamed CLK
- net /d0 renamed D0
- net /d1 renamed D1
- net /d2 renamed D2
- net /d3 renamed D3
- net /d4 renamed D4
- net /d5 renamed D5
- net /d6 renamed D6
- net /d7 renamed D7
- net /rx renamed UART_RX
- net /tx renamed UART_TX
- net /user1 renamed USER1
- net /user2 renamed USER2
- net /user3 renamed USER3
- net /~{busrq} renamed /~{BUSRQ}
- net /~{int} renamed ~{INT}
- net /~{iorq} renamed ~{IORQ}
- net /~{m1} renamed ~{M1}
- net /~{mreq} renamed ~{MREQ}
- net /~{nmi} renamed /~{NMI}
- net /~{rd} renamed ~{RD}
- net /~{reset} renamed ~{RESET}
- net /~{wait} renamed /~{WAIT}
- net /~{wr} renamed ~{WR}
Routing:
- net unconnected-(X1-NC-Pad1): track 7.62 -> 0.00 mm
- net ~{RESET}: track 32.2 -> 37.1 mm
- net VCC: track 324.6 -> 328.4 mm
- net /~{NMI}: track 29.5 -> 30.3 mm
- net /~{WAIT}: track 12.6 -> 13.3 mm
Other:
- board text added: "REV 2"
- board text added: "~{BRQ}"
- board text added: "~{NMI}"
- board text added: "~{RES}"
- board text added: "~{WAIT}"
- board text removed: "REV 1"
